File: McuSensorMotors.kicad_sch (KiCad schematic)
At the start: 1 part, among them U1 NUCLEO-G474RE

Commit message: Switched pins for SPI
Connections:
- net GPIO_Output_[Loop Timing 1]: now also U1.CN10_28 (PB14); no longer U1.CN10_26 (PB15)
- net SPI2_MISO: no longer U1.CN10_28 (PB14)
- new net SPI2_MOSI: U1.CN10_26 (PB15)
Changed lines of the file:
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@@
+		)
+	)
+	(label "GPIO_Output_[Loop Timing 1]"
+		(at 238.76 60.96 0)
+		(effects
+			(font
+				(size 1.27 1.27)
+			)
+			(justify left)
 		)
 	)
@@
 		)
 	)
-	(label "SPI2_MISO"
-		(at 238.76 60.96 0)
-		(effects
-			(font
-				(size 1.27 1.27)
-			)
-			(justify left)
-		)
-	)
 	(label "TIM1_CH3_[PWM]"
 		(at 185.42 95.25 180)
@@
 		)
 	)
-	(label "GPIO_Output_[Loop Timing 1]"
-		(at 238.76 58.42 0)
-		(effects
-			(font
-				(size 1.27 1.27)
-			)
-			(justify left)
-		)
-	)
 	(label "I2C2_SDA"
 		(at 177.8 55.88 180)
@@
 		(effects
 			(font
+				(size 1.27 1.27)
+			)
+			(justify left)
+		)
+	)
+	(label "SPI2_MOSI"
+		(at 238.76 58.42 0)
+		(effects
+			(font

Commit message: Changed some signal names
Connections:
- net GPIO_Output_[Loop Timing 3] is gone; now on net GPIO_Output_[Loop Timing 2]: U1.CN10_13 (PA6)
- net GPIO_Output_[Loop Timing 1]: now also U1.CN10_22 (PB2); no longer U1.CN10_28 (PB14)
- net GPIO_Output_[Loop Timing 2]: no longer U1.CN10_22 (PB2)
- new net GPIO_Output_[Loop Timing 0]: U1.CN10_28 (PB14)
Changed lines of the file:
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@@
 		)
 	)
-	(label "GPIO_Output_[Loop Timing 1]"
+	(label "GPIO_Output_[Loop Timing 0]"
 		(at 238.76 60.96 0)
 		(effects
@@
 		)
 	)
-	(label "GPIO_Output_[Loop Timing 2]"
+	(label "GPIO_Output_[Loop Timing 1]"
 		(at 238.76 53.34 0)
 		(effects
@@
 		)
 	)
-	(label "GPIO_Output_[Loop Timing 3]"
+	(label "GPIO_Output_[Loop Timing 2]"
 		(at 177.8 43.18 180)
 		(effects
